Commit message: added images and fixed box_height in pcb box (nano and motor driver, green box)

File: urdf/_jetbot.urdf (robot description, URDF)
Before this commit: robot jetbot, 28 links, 27 joints
Joints:
- joint base_nano_joint: origin xyz=0 0 0.035 -> xyz=0 0 0.055

File: urdf/jetbot.xacro (robot description, xacro)
@@ -452,5 +452,5 @@
     <parent link="base_link"/>
     <child link="pcb_boards"/>
-    <origin xyz="0 0 ${base_height}"/>
+    <origin xyz="0 0 ${box_height}"/>
   </joint>
   <!-- PCB, MOTOR DRIVER AND JETSON NANO -->
