Commit message: added gazebo plugins and controllers

File: urdf/jetbot.xacro (robot description, xacro)
@@ -61,7 +61,32 @@
     <inertial>
       <mass value="${mass}" />
-      <inertia ixx="1.0" ixy="0.0" ixz="0.0" iyy="1.0" iyz="0.0" izz="1.0" />
+      <inertia ixx="0.1" ixy="0.0" ixz="0.0" iyy="0.1" iyz="0.0" izz="0.1" />
     </inertial>
   </xacro:macro>
+  <!-- A simple inertial macro -->
+  <!-- transmission macro -->
+  <xacro:macro name="tx" params="prefix suffix">
+    <transmission name="${prefix}_${suffix}_trans">
+      <type>transmission_interface/SimpleTransmission</type>
+      <actuator name="${prefix}_${suffix}_motor">
+        <mechanicalReduction>1</mechanicalReduction>
+      </actuator>
+      <joint name="${prefix}_${suffix}_joint">
+        <hardwareInterface>hardware_interface/VelocityJointInterface</hardwareInterface>
+      </joint>
+    </transmission>
+  </xacro:macro>
+  <!-- transmission macro -->
+  <!-- pid macro -->
+  <!--xacro:macro name="pidctl" params="prefix suffix">
+    <gazebo reference="${prefix}_${suffix}">
+      <mu1 value="200.0"/>
+      <mu2 value="100.0"/>
+      <kp value="10000000.0" />
+      <kd value="1.0" />
+      <material>Gazebo/Grey</material>
+    </gazebo>
+  </xacro:macro-->
+  <!-- pid macro -->
   <!-- Wheel Macro-->
   <xacro:macro name="wheel_parts" params="prefix reflect">
@@ -80,5 +105,5 @@
       </geometry>
     </collision>
-    <xacro:inertia mass="1" />
+    <xacro:inertia mass="0.05" />
   </link>
   <joint name="base_${prefix}_wheel_shaft_joint" type="fixed">
@@ -102,5 +127,5 @@
       </geometry>
     </collision>
-    <xacro:inertia mass="1" />
+    <xacro:inertia mass="0.1" />
   </link>
   <joint name="${prefix}_shaft_wheelc_joint" type="fixed">
@@ -123,7 +148,7 @@
       </geometry>
     </collision>
-    <xacro:inertia mass="1" />
-  </link>
-  <joint name="${prefix}_wheelc_wheel_joint" type="continuous">
+    <xacro:inertia mass="0.1" />
+  </link>
+  <joint name="${prefix}_wheel_joint" type="continuous">
     <axis xyz="0 1 0"/>
     <parent link="${prefix}_wheelc"/>
@@ -131,4 +156,6 @@
     <origin xyz ="0 ${-0.0001*reflect} 0"/>
   </joint>
+  <!--xacro:pidctl prefix="${prefix}" suffix="wheel"/-->
+  <xacro:tx prefix="${prefix}" suffix="wheel" />
   </xacro:macro>
   <!-- Wheel Macro-->
@@ -147,5 +174,5 @@
       </geometry>
     </collision>
-    <xacro:inertia mass="1" />
+    <xacro:inertia mass="0.05" />
   </link>
   <joint name="${prefix}_caster_${suffix}_cyl_joint" type="fixed">
@@ -170,5 +197,5 @@
       </geometry>
     </collision>
-    <xacro:inertia mass="1" />
+    <xacro:inertia mass="0.05" />
   </link>
   <joint name="base_${prefix}_caster_joint" type="fixed">
@@ -179,5 +206,5 @@
   <xacro:caster_minicyl prefix="${prefix}" suffix="lt" reflect="1" />
   <xacro:caster_minicyl prefix="${prefix}" suffix="rt" reflect="-1" />
-  <link name="${prefix}_caster_ball">
+  <link name="${prefix}_caster">
     <visual>
       <geometry>
@@ -191,12 +218,14 @@
       </geometry>
     </collision>
-    <xacro:inertia mass="1" />
-  </link>
-  <joint name="${prefix}_caster_ball_joint" type="continuous">
+    <xacro:inertia mass="0.2" />
+  </link>
+  <joint name="${prefix}_caster_joint" type="continuous">
     <axis xyz="1 1 1" rpy="0 0 0" />
     <parent link="${prefix}_caster_base"/>
-    <child link="${prefix}_caster_ball"/>
+    <child link="${prefix}_caster"/>
     <origin xyz="0 0 -0.004"/>
   </joint>
+  <!--xacro:pidctl prefix="${prefix}" suffix="caster"/-->
+  <xacro:tx prefix="${prefix}" suffix="caster" />
   </xacro:macro>
   <!-- Left and Caster Wheel Macros, Including Mini Cylinders -->
@@ -217,5 +246,5 @@
       </geometry>
     </collision>
-    <xacro:inertia mass="1" />
+    <xacro:inertia mass="0.2" />
   </link>
   <joint name="base_${prefix}_antenna_joint" type="fixed">
@@ -236,5 +265,5 @@
       </geometry>
     </collision>
-    <xacro:inertia mass="1" />
+    <xacro:inertia mass="0.005" />
   </link>
   <joint name="${prefix}_antenna_top_joint" type="fixed">
@@ -260,5 +289,5 @@
       </geometry>
     </collision>
-    <xacro:inertia mass="1" />
+    <xacro:inertia mass="20" />
   </link>
   <!-- CHASSIS (body) -->
@@ -288,4 +317,5 @@
       </geometry>
     </collision>
+    <xacro:inertia mass="0.05" />
   </link>
   <joint name="camera_mount_base_joint" type="fixed">
@@ -308,4 +338,5 @@
       </geometry>
     </collision>
+    <xacro:inertia mass="0.05" />
   </link>
   <joint name="camera_mount_over_joint" type="fixed">
@@ -328,4 +359,5 @@
       </geometry>
     </collision>
+    <xacro:inertia mass="0.05" />
   </link>
   <joint name="camera_mount_angled_joint" type="fixed">
@@ -348,4 +380,5 @@
       </geometry>
     </collision>
+    <xacro:inertia mass="0.05" />
   </link>
   <joint name="camera_mount_screen_joint" type="fixed">
@@ -368,4 +401,5 @@
       </geometry>
     </collision>
+    <xacro:inertia mass="0.05" />
   </link>
   <joint name="camera_pcb_base_joint" type="fixed">
@@ -388,4 +422,5 @@
       </geometry>
     </collision>
+    <xacro:inertia mass="0.05" />
   </link>
   <joint name="camera_lens_body_joint" type="fixed">
@@ -408,4 +443,5 @@
       </geometry>
     </collision>
+    <xacro:inertia mass="0.05" />
   </link>
  <joint name="camera_lens_body_out_joint" type="fixed">
@@ -428,4 +464,5 @@
       </geometry>
     </collision>
+    <xacro:inertia mass="0.05" />
   </link>
  <joint name="camera_lens_joint" type="fixed">
@@ -447,5 +484,5 @@
       </geometry>
     </collision>
-    <xacro:inertia mass="1" />
+    <xacro:inertia mass="20" />
   </link>
   <joint name="base_nano_joint" type="fixed">
@@ -455,3 +492,9 @@
   </joint>
   <!-- PCB, MOTOR DRIVER AND JETSON NANO -->
+  <!-- Gazebo plugin for ROS Control -->
+  <gazebo>
+    <plugin name="gazebo_ros_control" filename="libgazebo_ros_control.so">
+      <robotNamespace>/</robotNamespace>
+    </plugin>
+  </gazebo>
 </robot>

Commit message: fixed physics and pid a little (pure p control) with help of Lentin

File: urdf/jetbot.xacro (robot description, xacro)
@@ -1,3 +1,8 @@
 <?xml version="1.0"?>
+<!-- Inertia Equations -->
+<!-- https://bit.ly/2S0aK32 -->
+<!-- ixx ixy ixz -->
+<!-- ixy iyy iyz -->
+<!-- ixz iyz izz -->
 <robot xmlns:xacro="http://www.ros.org/wiki/xacro" name="jetbot">
   <!-- Chassis constants -->
@@ -20,5 +25,5 @@
   <xacro:property name="caster_xoffset" value="0.06" />
   <xacro:property name="caster_yoffset" value="0.008" />
-  <xacro:property name="caster_zoffset" value="-0.01" />
+  <xacro:property name="caster_zoffset" value="-0.0097" />
   <xacro:property name="caster_ball" value="0.005" />
   <!-- Caster Ball constants -->
@@ -60,9 +65,28 @@
   <xacro:macro name="inertia" params="mass">
     <inertial>
-      <mass value="${mass}" />
-      <inertia ixx="0.1" ixy="0.0" ixz="0.0" iyy="0.1" iyz="0.0" izz="0.1" />
+      <mass value="${mass}"/>
+      <inertia ixx="0.01" ixy="0.0" ixz="0.0" iyy="0.01" iyz="0.0" izz="0.01"/>
     </inertial>
   </xacro:macro>
   <!-- A simple inertial macro -->
+  <!-- cuboid inertia -->
+  <xacro:macro name="cuboid_inertia" params="mass x y z">
+      <inertia  ixx="${mass*(y*y+z*z)/12}" ixy = "0" ixz = "0"
+                iyy="${mass*(x*x+z*z)/12}" iyz = "0"
+                izz="${mass*(x*x+z*z)/12}" />
+  </xacro:macro>
+  <!-- cuboid inertia -->
+  <!-- sphere inertia -->
+  <xacro:macro name="sphere_inertia" params="mass r">
+    <inertia  ixx="${2*mass*r*r/5}" ixy = "0" ixz = "0"
+              iyy="${2*mass*r*r/5}" iyz = "0"
+              izz="${2*mass*r*r/5}" />
+  </xacro:macro>
+  <!-- sphere inertia -->
+  <xacro:macro name="cylinder_inertia" params="mass r h">
+    <inertia  ixx="${mass*(3*r*r+h*h)/12}" ixy = "0" ixz = "0"
+              iyy="${mass*(3*r*r+h*h)/12}" iyz = "0"
+              izz="${mass*r*r/2}" />
+  </xacro:macro>
   <!-- transmission macro -->
   <xacro:macro name="tx" params="prefix suffix">
@@ -78,15 +102,4 @@
   </xacro:macro>
   <!-- transmission macro -->
-  <!-- pid macro -->
-  <!--xacro:macro name="pidctl" params="prefix suffix">
-    <gazebo reference="${prefix}_${suffix}">
-      <mu1 value="200.0"/>
-      <mu2 value="100.0"/>
-      <kp value="10000000.0" />
-      <kd value="1.0" />
-      <material>Gazebo/Grey</material>
-    </gazebo>
-  </xacro:macro-->
-  <!-- pid macro -->
   <!-- Wheel Macro-->
   <xacro:macro name="wheel_parts" params="prefix reflect">
@@ -105,5 +118,5 @@
       </geometry>
     </collision>
-    <xacro:inertia mass="0.05" />
+    <xacro:inertia mass="0.6" />
   </link>
   <joint name="base_${prefix}_wheel_shaft_joint" type="fixed">
@@ -127,5 +140,5 @@
       </geometry>
     </collision>
-    <xacro:inertia mass="0.1" />
+    <xacro:inertia mass="0.6" />
   </link>
   <joint name="${prefix}_shaft_wheelc_joint" type="fixed">
@@ -148,5 +161,5 @@
       </geometry>
     </collision>
-    <xacro:inertia mass="0.1" />
+    <xacro:inertia mass="0.6" />
   </link>
   <joint name="${prefix}_wheel_joint" type="continuous">
@@ -156,5 +169,4 @@
     <origin xyz ="0 ${-0.0001*reflect} 0"/>
   </joint>
-  <!--xacro:pidctl prefix="${prefix}" suffix="wheel"/-->
   <xacro:tx prefix="${prefix}" suffix="wheel" />
   </xacro:macro>
@@ -174,5 +186,5 @@
       </geometry>
     </collision>
-    <xacro:inertia mass="0.05" />
+    <xacro:inertia mass="0.6" />
   </link>
   <joint name="${prefix}_caster_${suffix}_cyl_joint" type="fixed">
@@ -197,5 +209,5 @@
       </geometry>
     </collision>
-    <xacro:inertia mass="0.05" />
+    <xacro:inertia mass="0.6" />
   </link>
   <joint name="base_${prefix}_caster_joint" type="fixed">
@@ -218,14 +230,14 @@
       </geometry>
     </collision>
-    <xacro:inertia mass="0.2" />
-  </link>
-  <joint name="${prefix}_caster_joint" type="continuous">
-    <axis xyz="1 1 1" rpy="0 0 0" />
+    <xacro:inertia mass="0.6" />
+  </link>
+  <joint name="${prefix}_caster_joint" type="fixed">
+  <!--joint name="${prefix}_caster_joint" type="continuous">
+    <axis xyz="1 1 1" rpy="0 0 0" /-->
     <parent link="${prefix}_caster_base"/>
     <child link="${prefix}_caster"/>
     <origin xyz="0 0 -0.004"/>
   </joint>
-  <!--xacro:pidctl prefix="${prefix}" suffix="caster"/-->
-  <xacro:tx prefix="${prefix}" suffix="caster" />
+  <!--xacro:tx prefix="${prefix}" suffix="caster" /-->
   </xacro:macro>
   <!-- Left and Caster Wheel Macros, Including Mini Cylinders -->
@@ -246,5 +258,5 @@
       </geometry>
     </collision>
-    <xacro:inertia mass="0.2" />
+    <xacro:inertia mass="0.6" />
   </link>
   <joint name="base_${prefix}_antenna_joint" type="fixed">
@@ -265,5 +277,5 @@
       </geometry>
     </collision>
-    <xacro:inertia mass="0.005" />
+    <xacro:inertia mass="0.06" />
   </link>
   <joint name="${prefix}_antenna_top_joint" type="fixed">
@@ -289,5 +301,5 @@
       </geometry>
     </collision>
-    <xacro:inertia mass="20" />
+    <xacro:inertia mass="0.6" />
   </link>
   <!-- CHASSIS (body) -->
@@ -317,5 +329,5 @@
       </geometry>
     </collision>
-    <xacro:inertia mass="0.05" />
+    <xacro:inertia mass="0.6" />
   </link>
   <joint name="camera_mount_base_joint" type="fixed">
@@ -338,5 +350,5 @@
       </geometry>
     </collision>
-    <xacro:inertia mass="0.05" />
+    <xacro:inertia mass="0.6" />
   </link>
   <joint name="camera_mount_over_joint" type="fixed">
@@ -359,5 +371,5 @@
       </geometry>
     </collision>
-    <xacro:inertia mass="0.05" />
+    <xacro:inertia mass="0.6" />
   </link>
   <joint name="camera_mount_angled_joint" type="fixed">
@@ -380,5 +392,5 @@
       </geometry>
     </collision>
-    <xacro:inertia mass="0.05" />
+    <xacro:inertia mass="0.6" />
   </link>
   <joint name="camera_mount_screen_joint" type="fixed">
@@ -401,5 +413,5 @@
       </geometry>
     </collision>
-    <xacro:inertia mass="0.05" />
+    <xacro:inertia mass="0.6" />
   </link>
   <joint name="camera_pcb_base_joint" type="fixed">
@@ -422,5 +434,5 @@
       </geometry>
     </collision>
-    <xacro:inertia mass="0.05" />
+    <xacro:inertia mass="0.6" />
   </link>
   <joint name="camera_lens_body_joint" type="fixed">
@@ -443,5 +455,5 @@
       </geometry>
     </collision>
-    <xacro:inertia mass="0.05" />
+    <xacro:inertia mass="0.6" />
   </link>
  <joint name="camera_lens_body_out_joint" type="fixed">
@@ -464,5 +476,5 @@
       </geometry>
     </collision>
-    <xacro:inertia mass="0.05" />
+    <xacro:inertia mass="0.6" />
   </link>
  <joint name="camera_lens_joint" type="fixed">
@@ -484,5 +496,5 @@
       </geometry>
     </collision>
-    <xacro:inertia mass="20" />
+    <xacro:inertia mass="0.6" />
   </link>
   <joint name="base_nano_joint" type="fixed">

Commit message: fixed inertias, match a lower number if you have problems, now the model moves straight

File: urdf/jetbot.xacro (robot description, xacro)
@@ -66,5 +66,5 @@
     <inertial>
       <mass value="${mass}"/>
-      <inertia ixx="0.01" ixy="0.0" ixz="0.0" iyy="0.01" iyz="0.0" izz="0.01"/>
+      <inertia ixx="0.04" ixy="0.0" ixz="0.0" iyy="0.04" iyz="0.0" izz="0.04"/>
     </inertial>
   </xacro:macro>
@@ -161,5 +161,5 @@
       </geometry>
     </collision>
-    <xacro:inertia mass="0.6" />
+    <xacro:inertia mass="0.6"/>
   </link>
   <joint name="${prefix}_wheel_joint" type="continuous">
@@ -186,5 +186,5 @@
       </geometry>
     </collision>
-    <xacro:inertia mass="0.6" />
+    <xacro:cylinder_inertia mass="0.6" r="${caster_cyl_r/3.75}" h="${caster_cyl_len}" />
   </link>
   <joint name="${prefix}_caster_${suffix}_cyl_joint" type="fixed">
@@ -209,5 +209,5 @@
       </geometry>
     </collision>
-    <xacro:inertia mass="0.6" />
+    <xacro:cylinder_inertia mass="0.6" r="${caster_cyl_r}" h="${caster_cyl_len}" />
   </link>
   <joint name="base_${prefix}_caster_joint" type="fixed">
@@ -230,5 +230,5 @@
       </geometry>
     </collision>
-    <xacro:inertia mass="0.6" />
+    <xacro:sphere_inertia mass="0.6" r="${caster_ball}" />
   </link>
   <joint name="${prefix}_caster_joint" type="fixed">
@@ -258,5 +258,5 @@
       </geometry>
     </collision>
-    <xacro:inertia mass="0.6" />
+    <xacro:cylinder_inertia mass="0.6" r="${antenna_r}" h="${antenna_len}" />
   </link>
   <joint name="base_${prefix}_antenna_joint" type="fixed">
@@ -277,5 +277,5 @@
       </geometry>
     </collision>
-    <xacro:inertia mass="0.06" />
+    <xacro:sphere_inertia mass="0.06" r="${antenna_r}" />
   </link>
   <joint name="${prefix}_antenna_top_joint" type="fixed">
@@ -301,5 +301,5 @@
       </geometry>
     </collision>
-    <xacro:inertia mass="0.6" />
+    <xacro:cuboid_inertia mass="0.6" x="${base_len}" y="${base_width}" z="${base_height}" />
   </link>
   <!-- CHASSIS (body) -->
@@ -329,5 +329,5 @@
       </geometry>
     </collision>
-    <xacro:inertia mass="0.6" />
+    <xacro:cuboid_inertia mass="0.6" x="0.01" y="0.04" z="0.002" />
   </link>
   <joint name="camera_mount_base_joint" type="fixed">
@@ -350,5 +350,5 @@
       </geometry>
     </collision>
-    <xacro:inertia mass="0.6" />
+    <xacro:cuboid_inertia mass="0.6" x="0.03" y="0.04" z="0.002"/>
   </link>
   <joint name="camera_mount_over_joint" type="fixed">
@@ -371,5 +371,5 @@
       </geometry>
     </collision>
-    <xacro:inertia mass="0.6" />
+    <xacro:cuboid_inertia mass="0.6" x="0.025" y="0.025" z="0.002" />
   </link>
   <joint name="camera_mount_angled_joint" type="fixed">
@@ -392,5 +392,5 @@
       </geometry>
     </collision>
-    <xacro:inertia mass="0.6" />
+    <xacro:cuboid_inertia mass="0.6" x="0.025" y="0.025" z="0.004" />
   </link>
   <joint name="camera_mount_screen_joint" type="fixed">
@@ -413,5 +413,5 @@
       </geometry>
     </collision>
-    <xacro:inertia mass="0.6" />
+    <xacro:cuboid_inertia mass="0.6" x="0.013" y="0.013" z="0.004" />
   </link>
   <joint name="camera_pcb_base_joint" type="fixed">
@@ -434,5 +434,5 @@
       </geometry>
     </collision>
-    <xacro:inertia mass="0.6" />
+    <xacro:cylinder_inertia mass="0.6" r="0.006" h="0.01" />
   </link>
   <joint name="camera_lens_body_joint" type="fixed">
@@ -455,5 +455,5 @@
       </geometry>
     </collision>
-    <xacro:inertia mass="0.6" />
+    <xacro:cylinder_inertia mass="0.6" r="0.0075" h="0.003"/>
   </link>
  <joint name="camera_lens_body_out_joint" type="fixed">
@@ -476,5 +476,5 @@
       </geometry>
     </collision>
-    <xacro:inertia mass="0.6" />
+    <xacro:sphere_inertia mass="0.6" r="0.005" />
   </link>
  <joint name="camera_lens_joint" type="fixed">
@@ -496,5 +496,5 @@
       </geometry>
     </collision>
-    <xacro:inertia mass="0.6" />
+    <xacro:cuboid_inertia mass="0.6" x="${box_len}" y="${box_width}" z="${box_height}" />
   </link>
   <joint name="base_nano_joint" type="fixed">
