Commit message: added camera plugin and separate xacro in several includes

File: urdf/jetbot.xacro (robot description, xacro)
@@ -1,307 +1,9 @@
 <?xml version="1.0"?>
-<!-- Inertia Equations -->
-<!-- https://bit.ly/2S0aK32 -->
-<!-- ixx ixy ixz -->
-<!-- ixy iyy iyz -->
-<!-- ixz iyz izz -->
 <robot xmlns:xacro="http://www.ros.org/wiki/xacro" name="jetbot">
-  <!-- Chassis constants -->
-  <xacro:property name="base_len" value="0.134"/>
-  <xacro:property name="base_width" value="0.095"/>
-  <xacro:property name="base_height" value="0.035"/>
-  <xacro:property name="base_z_offset" value="0.013"/>
-  <!-- Chassis constants -->
-  <!-- Wheel constants -->
-  <xacro:property name="shaft_len" value="0.015" />
-  <xacro:property name="shaft_r" value="0.005" />
-  <xacro:property name="shaft_xoffset" value="0.023" />
-  <xacro:property name="shaft_yoffset" value="0.048" />
-  <xacro:property name="wheelc_len" value="0.015" />
-  <xacro:property name="wheelc_r" value = "0.026" />
-  <!-- Wheel constants -->
-  <!-- Caster Ball constants -->
-  <xacro:property name="caster_cyl_len" value="0.01" />
-  <xacro:property name="caster_cyl_r" value="0.0075" />
-  <xacro:property name="caster_xoffset" value="0.06" />
-  <xacro:property name="caster_yoffset" value="0.008" />
-  <xacro:property name="caster_zoffset" value="-0.0097" />
-  <xacro:property name="caster_ball" value="0.005" />
-  <!-- Caster Ball constants -->
-  <!-- Antenna constants -->
-  <xacro:property name="antenna_len" value="0.19" />
-  <xacro:property name="antenna_r" value="0.005" />
-  <xacro:property name="antenna_x" value="-0.645" />
-  <!-- Antenna constants -->
-  <!-- Motor driver and PCB constants -->
-  <xacro:property name="box_len" value="0.105" />
-  <xacro:property name="box_width" value="0.08" />
-  <xacro:property name="box_height" value="0.055" />
-  <!-- Motor driver and PCB constants -->
-  <!-- Color Properties -->
-  <material name="black">
-    <color rgba="0 0 0 1"/>
-  </material>
-  <material name="white">
-    <color rgba="1.0 1.0 1.0 1.0"/>
-  </material>
-  <material name="blue">
-    <color rgba="0 0 1 0.2"/>
-  </material>
-  <material name="grey">
-    <color rgba="0.66 0.66 0.66 1"/>
-  </material>
-  <material name="soft_blue">
-    <color rgba="0.2157 0.5294 0.9216 1"/>
-  </material>
-  <material name="grey_alpha">
-    <color rgba="0.3 0.3 0.3 0.4"/>
-  </material>
-  <material name="green">
-    <color rgba="0.1 0.3 0.1 0.8"/>
-  </material>
-  <!-- Color Properties -->
-  <!-- Xacro Macros -->
-  <!-- A simple inertial macro -->
-  <xacro:macro name="inertia" params="mass">
-    <inertial>
-      <mass value="${mass}"/>
-      <inertia ixx="0.04" ixy="0.0" ixz="0.0" iyy="0.04" iyz="0.0" izz="0.04"/>
-    </inertial>
-  </xacro:macro>
-  <!-- A simple inertial macro -->
-  <!-- cuboid inertia -->
-  <xacro:macro name="cuboid_inertia" params="mass x y z">
-      <inertia  ixx="${mass*(y*y+z*z)/12}" ixy = "0" ixz = "0"
-                iyy="${mass*(x*x+z*z)/12}" iyz = "0"
-                izz="${mass*(x*x+z*z)/12}" />
-  </xacro:macro>
-  <!-- cuboid inertia -->
-  <!-- sphere inertia -->
-  <xacro:macro name="sphere_inertia" params="mass r">
-    <inertia  ixx="${2*mass*r*r/5}" ixy = "0" ixz = "0"
-              iyy="${2*mass*r*r/5}" iyz = "0"
-              izz="${2*mass*r*r/5}" />
-  </xacro:macro>
-  <!-- sphere inertia -->
-  <xacro:macro name="cylinder_inertia" params="mass r h">
-    <inertia  ixx="${mass*(3*r*r+h*h)/12}" ixy = "0" ixz = "0"
-              iyy="${mass*(3*r*r+h*h)/12}" iyz = "0"
-              izz="${mass*r*r/2}" />
-  </xacro:macro>
-  <!-- transmission macro -->
-  <xacro:macro name="tx" params="prefix suffix">
-    <transmission name="${prefix}_${suffix}_trans">
-      <type>transmission_interface/SimpleTransmission</type>
-      <actuator name="${prefix}_${suffix}_motor">
-        <mechanicalReduction>1</mechanicalReduction>
-      </actuator>
-      <joint name="${prefix}_${suffix}_joint">
-        <hardwareInterface>hardware_interface/VelocityJointInterface</hardwareInterface>
-      </joint>
-    </transmission>
-  </xacro:macro>
-  <!-- transmission macro -->
-  <!-- Wheel Macro-->
-  <xacro:macro name="wheel_parts" params="prefix reflect">
-  <link name="${prefix}_wheel_shaft">
-    <visual>
-      <origin xyz="0 0 0" rpy="${pi/2} 0 0"/>
-      <geometry>
-        <cylinder radius="${shaft_r}" length="${shaft_len}" />
-      </geometry>
-      <material name="white"/>
-    </visual>
-    <collision>
-      <origin xyz="0 0 0" rpy="${pi/2} 0 0"/>
-      <geometry>
-        <cylinder radius="${shaft_r}" length="${shaft_len}" />
-      </geometry>
-    </collision>
-    <xacro:inertia mass="0.6" />
-  </link>
-  <joint name="base_${prefix}_wheel_shaft_joint" type="fixed">
-    <axis rpy="0 0 0" xyz="0 0 0" />
-    <parent link="base_link"/>
-    <child link="${prefix}_wheel_shaft"/>
-    <origin rpy="0 0 0" xyz="${shaft_xoffset} ${shaft_yoffset*reflect} 0.013" />
-  </joint>
-  <link name="${prefix}_wheelc">
-    <visual>
-      <origin rpy="${pi/2} 0 0"/>
-      <geometry>
-        <cylinder length="${wheelc_len}" radius="${wheelc_r}"/>
-      </geometry>
-      <material name="white"/>
-    </visual>
-    <collision>
-      <origin rpy="${pi/2} 0 0"/>
-      <geometry>
-        <cylinder length="${wheelc_len}" radius="${wheelc_r}"/>
-      </geometry>
-    </collision>
-    <xacro:inertia mass="0.6" />
-  </link>
-  <joint name="${prefix}_shaft_wheelc_joint" type="fixed">
-    <origin xyz="0 ${reflect*(wheelc_r-0.002)/2} 0"/>
-    <parent link="${prefix}_wheel_shaft"/>
-    <child link="${prefix}_wheelc"/>
-  </joint>
-  <link name="${prefix}_wheel">
-    <visual>
-    <origin rpy="${pi/2} 0 0" xyz="0 0 0" />
-      <geometry>
-        <cylinder length="${wheelc_len}" radius="${wheelc_r + 0.0065}"/>
-      </geometry>
-      <material name="black"/>
-    </visual>
-    <collision>
-    <origin rpy="${pi/2} 0 0" xyz="0 0 0" />
-      <geometry>
-        <cylinder length="${wheelc_len}" radius="${wheelc_r + 0.0065}"/>
-      </geometry>
-    </collision>
-    <xacro:inertia mass="0.6"/>
-  </link>
-  <joint name="${prefix}_wheel_joint" type="continuous">
-    <axis xyz="0 1 0"/>
-    <parent link="${prefix}_wheelc"/>
-    <child link="${prefix}_wheel"/>
-    <origin xyz ="0 ${-0.0001*reflect} 0"/>
-  </joint>
-  <xacro:tx prefix="${prefix}" suffix="wheel" />
-  </xacro:macro>
-  <!-- Wheel Macro-->
-  <!-- Caster Wheel Left and Right Mini Cylinder Macros -->
-  <xacro:macro name="caster_minicyl" params="prefix suffix reflect">
-  <link name="${prefix}_caster_${suffix}_cyl">
-    <visual>
-      <geometry>
-        <cylinder length="${caster_cyl_len}" radius="${caster_cyl_r/3.75}"/>
-      </geometry>
-      <material name="white"/>
-    </visual>
-    <collision>
-      <geometry>
-        <cylinder length="${caster_cyl_len}" radius="${caster_cyl_r/3.75}"/>
-      </geometry>
-    </collision>
-    <xacro:cylinder_inertia mass="0.6" r="${caster_cyl_r/3.75}" h="${caster_cyl_len}" />
-  </link>
-  <joint name="${prefix}_caster_${suffix}_cyl_joint" type="fixed">
-    <origin xyz="0 ${reflect*caster_yoffset} 0"/>
-    <parent link="${prefix}_caster_base"/>
-    <child link="${prefix}_caster_${suffix}_cyl"/>
-  </joint>
-  </xacro:macro>
-  <!-- Caster Wheel Left and Right Mini Cylinder Macros -->
-  <!-- Left and Caster Wheel Macros, Including Mini Cylinders -->
-  <xacro:macro name="caster_wheel_parts" params="prefix reflect">
-  <link name="${prefix}_caster_base">
-    <visual>
-      <geometry>
-        <cylinder length="${caster_cyl_len}" radius="${caster_cyl_r}"/>
-      </geometry>
-      <material name="white"/>
-    </visual>
-    <collision>
-      <geometry>
-        <cylinder length="${caster_cyl_len}" radius="${caster_cyl_r}"/>
-      </geometry>
-    </collision>
-    <xacro:cylinder_inertia mass="0.6" r="${caster_cyl_r}" h="${caster_cyl_len}" />
-  </link>
-  <joint name="base_${prefix}_caster_joint" type="fixed">
-    <origin xyz="${reflect*caster_xoffset} 0 ${caster_zoffset}"/>
-    <parent link="base_link"/>
-    <child link="${prefix}_caster_base"/>
-  </joint>
-  <xacro:caster_minicyl prefix="${prefix}" suffix="lt" reflect="1" />
-  <xacro:caster_minicyl prefix="${prefix}" suffix="rt" reflect="-1" />
-  <link name="${prefix}_caster">
-    <visual>
-      <geometry>
-        <sphere radius="${caster_ball}" />
-      </geometry>
-      <material name="grey"/>
-    </visual>
-    <collision>
-      <geometry>
-        <sphere radius="${caster_ball}" />
-      </geometry>
-    </collision>
-    <xacro:sphere_inertia mass="0.6" r="${caster_ball}" />
-  </link>
-  <joint name="${prefix}_caster_joint" type="fixed">
-  <!--joint name="${prefix}_caster_joint" type="continuous">
-    <axis xyz="1 1 1" rpy="0 0 0" /-->
-    <parent link="${prefix}_caster_base"/>
-    <child link="${prefix}_caster"/>
-    <origin xyz="0 0 -0.004"/>
-  </joint>
-  <!--xacro:tx prefix="${prefix}" suffix="caster" /-->
-  </xacro:macro>
-  <!-- Left and Caster Wheel Macros, Including Mini Cylinders -->
-  <!-- Left and Right Antenna Macro -->
-  <xacro:macro name="antenna" params="prefix reflect">
-  <link name="${prefix}_antenna">
-    <visual>
-      <origin xyz="0 0 ${antenna_len/2}"/>
-      <geometry>
-        <cylinder length="${antenna_len}" radius="${antenna_r}"/>
-      </geometry>
-      <material name="black"/>
-    </visual>
-    <collision>
-      <origin xyz="0 0 ${antenna_len/2}"/>
-      <geometry>
-        <cylinder length="${antenna_len}" radius="${antenna_r}"/>
-      </geometry>
-    </collision>
-    <xacro:cylinder_inertia mass="0.6" r="${antenna_r}" h="${antenna_len}" />
-  </link>
-  <joint name="base_${prefix}_antenna_joint" type="fixed">
-    <parent link="base_link"/>
-    <child link="${prefix}_antenna"/>
-    <origin xyz="-${(base_len/2 - antenna_r)} ${reflect*(antenna_r + 0.0375)} 0.0305"/>
-  </joint>
-  <link name="${prefix}_antenna_top">
-    <visual>
-      <geometry>
-        <sphere radius="${antenna_r}"/>
-      </geometry>
-      <material name="black"/>
-    </visual>
-    <collision>
-      <geometry>
-        <sphere radius="${antenna_r}"/>
-      </geometry>
-    </collision>
-    <xacro:sphere_inertia mass="0.06" r="${antenna_r}" />
-  </link>
-  <joint name="${prefix}_antenna_top_joint" type="fixed">
-    <origin xyz="0 0 ${antenna_len}"/>
-    <parent link="${prefix}_antenna"/>
-    <child link="${prefix}_antenna_top"/>
-  </joint>
-  </xacro:macro>
-  <!-- Left and Right Antenna Macro -->
-  <!-- CHASSIS (body) -->
-  <link name="base_link">
-    <visual>
-      <origin xyz="0 0 ${base_z_offset}"/>
-      <geometry>
-        <box size="${base_len} ${base_width} ${base_height}"/>
-      </geometry>
-      <material name="blue"/>
-    </visual>
-    <collision>
-      <origin xyz="0 0 ${base_z_offset}"/>
-      <geometry>
-        <box size="${base_len} ${base_width} ${base_height}"/>
-      </geometry>
-    </collision>
-    <xacro:cuboid_inertia mass="0.6" x="${base_len}" y="${base_width}" z="${base_height}" />
-  </link>
-  <!-- CHASSIS (body) -->
+  <!-- All Neccesary Header Files, Macros and Constants -->
+  <xacro:include filename="$(find jetbot_diff_drive)/urdf/includes.xacro" />
+  <!-- All Neccesary Header FIles, Macros and Constants -->
+  <!-- CHASSIS -->
+  <xacro:include filename="$(find jetbot_diff_drive)/urdf/includes/parts/chassis.xacro" />
   <!-- LEFT WHEEL -->
   <xacro:wheel_parts prefix="lt" reflect="1" />
@@ -316,197 +18,7 @@
   <!-- RIGHT ANTENNA -->
   <xacro:antenna prefix="rt" reflect="-1" />
-<!-- CAMERA -->
-  <link name="camera_mount_base">
-    <visual>
-      <geometry>
-        <box size="0.01 0.04 0.002"/>
-      </geometry>
-      <material name="blue"/>
-    </visual>
-    <collision>
-      <geometry>
-        <box size="0.01 0.04 0.002"/>
-      </geometry>
-    </collision>
-    <xacro:cuboid_inertia mass="0.6" x="0.01" y="0.04" z="0.002" />
-  </link>
-  <joint name="camera_mount_base_joint" type="fixed">
-    <parent link="base_link"/>
-    <child link="camera_mount_base"/>
-    <origin rpy="0 0 0" xyz="0.0615 0 0.0315"/>
-  </joint>
-  <link name="camera_mount_over">
-    <visual>
-      <origin rpy="0 1.57079632679 0"/>
-      <geometry>
-        <box size="0.03 0.04 0.002"/>
-      </geometry>
-      <material name="blue"/>
-    </visual>
-    <collision>
-      <origin rpy="0 1.57079632679 0"/>
-      <geometry>
-        <box size="0.03 0.04 0.002"/>
-      </geometry>
-    </collision>
-    <xacro:cuboid_inertia mass="0.6" x="0.03" y="0.04" z="0.002"/>
-  </link>
-  <joint name="camera_mount_over_joint" type="fixed">
-    <parent link="camera_mount_base"/>
-    <child link="camera_mount_over"/>
-    <origin xyz="0.004 0 0.016"/>
-  </joint>
-  <link name="camera_mount_angled">
-    <visual>
-      <origin rpy="0 1.57079632679 0"/>
-      <geometry>
-        <box size="0.025 0.025 0.002"/>
-      </geometry>
-      <material name="blue"/>
-    </visual>
-    <collision>
-      <origin rpy="0 1.57079632679 0"/>
-      <geometry>
-        <box size="0.025 0.025 0.002"/>
-      </geometry>
-    </collision>
-    <xacro:cuboid_inertia mass="0.6" x="0.025" y="0.025" z="0.002" />
-  </link>
-  <joint name="camera_mount_angled_joint" type="fixed">
-    <parent link="camera_mount_over"/>
-    <child link="camera_mount_angled"/>
-    <origin rpy="0 0.463647609 0" xyz="0.0055 0 0.025"/>
-  </joint>
-  <link name="camera_screen_base">
-    <visual>
-      <origin rpy="0 1.57079632679 0"/>
-      <geometry>
-        <box size="0.025 0.025 0.004"/>
-      </geometry>
-      <material name="soft_blue"/>
-    </visual>
-    <collision>
-      <origin rpy="0 1.57079632679 0"/>
-      <geometry>
-        <box size="0.025 0.025 0.004"/>
-      </geometry>
-    </collision>
-    <xacro:cuboid_inertia mass="0.6" x="0.025" y="0.025" z="0.004" />
-  </link>
-  <joint name="camera_mount_screen_joint" type="fixed">
-    <parent link="camera_mount_angled"/>
-    <child link="camera_screen_base"/>
-    <origin rpy="0 0 0" xyz="0.0025 0 0"/>
-  </joint>
-  <link name="camera_pcb_base">
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