Commit message: added intel realsense D435 depth camera via xacro files

File: urdf/includes.xacro (robot description, xacro)
@@ -5,5 +5,5 @@
   <!-- Rviz Color Properties -->
   <!-- Gazebo Properties -->
-  <xacro:include filename="$(find jetbot_diff_drive)/urdf/includes/gazebo/jetbot.gazebo" />
+  <xacro:include filename="$(find jetbot_diff_drive)/urdf/includes/gazebo/jetbot.gazebo.xacro" />
   <!-- Gazebo Properties -->
   <!-- Transmission Macro -->
@@ -13,4 +13,7 @@
   <xacro:include filename="$(find jetbot_diff_drive)/urdf/includes/gazebo/inertias.xacro" />
   <!-- Inertia Macros -->
+  <!-- Chassis macro -->
+  <xacro:include filename="$(find jetbot_diff_drive)/urdf/includes/parts/chassis.xacro" />
+  <!-- Chassis macro -->
   <!-- Antenna Macro -->
   <xacro:include filename="$(find jetbot_diff_drive)/urdf/includes/parts/antenna.xacro" />
@@ -22,3 +25,12 @@
   <xacro:include filename="$(find jetbot_diff_drive)/urdf/includes/parts/wheels/caster.xacro" />
   <!-- Caster Wheel Macro -->
+  <!-- Camera-->
+  <xacro:include filename="$(find jetbot_diff_drive)/urdf/includes/parts/sensors/rgbcam/camera.xacro" />
+  <!-- Camera-->
+  <!-- PCB Boards -->
+  <xacro:include filename="$(find jetbot_diff_drive)/urdf/includes/parts/boards.xacro" />
+  <!-- PCB Boards -->
+  <!-- Intel Realsense Macro -->
+  <xacro:include filename="$(find jetbot_diff_drive)/urdf/includes/parts/sensors/realsense/_d435.urdf.xacro" />
+  <!-- Intel Realsense Macro -->
 </robot>

File: urdf/includes/parts/boards.xacro (robot description, xacro)
@@ -10,4 +10,5 @@
   <!-- Inertias Macros -->
   <!-- PCB, MOTOR DRIVER AND JETSON NANO -->
+  <xacro:macro name="pcb">
   <link name="pcb_boards">
     <visual>
@@ -29,4 +30,5 @@
     <origin xyz="0 0 ${box_height}"/>
   </joint>
+  </xacro:macro>
   <!-- PCB, MOTOR DRIVER AND JETSON NANO -->
 </robot>

File: urdf/includes/parts/chassis.xacro (robot description, xacro)
@@ -8,4 +8,5 @@
   <!-- Chassis constants -->
   <!-- CHASSIS (body) -->
+  <xacro:macro name="chassis" >
   <link name="base_link">
     <visual>
@@ -24,4 +25,5 @@
     <xacro:cuboid_inertia mass="0.6" x="${base_len}" y="${base_width}" z="${base_height}" />
   </link>
+  </xacro:macro>
   <!-- CHASSIS (body) -->
 </robot>

File: urdf/jetbot.xacro (robot description, xacro)
@@ -1,9 +1,12 @@
 <?xml version="1.0"?>
 <robot xmlns:xacro="http://www.ros.org/wiki/xacro" name="jetbot">
+  <!-- Xacro arguments for nominal use -->
+  <xacro:arg name="realsense_enable" default="true" />
+  <xacro:arg name="pointcloud_enable" default="true" />
   <!-- All Neccesary Header Files, Macros and Constants -->
   <xacro:include filename="$(find jetbot_diff_drive)/urdf/includes.xacro" />
   <!-- All Neccesary Header FIles, Macros and Constants -->
   <!-- CHASSIS -->
-  <xacro:include filename="$(find jetbot_diff_drive)/urdf/includes/parts/chassis.xacro" />
+  <xacro:chassis />
   <!-- LEFT WHEEL -->
   <xacro:wheel_parts prefix="lt" reflect="1" />
@@ -18,7 +21,14 @@
   <!-- RIGHT ANTENNA -->
   <xacro:antenna prefix="rt" reflect="-1" />
-  <!-- CAMERA -->
-  <xacro:include filename="$(find jetbot_diff_drive)/urdf/includes/parts/camera.xacro" />
+  <!-- SENSORS -->
+  <!-- MONOCULAR CAMERA -->
+  <xacro:camera />
+  <!-- REALSENSE CAMERA -->
+  <xacro:if value="$(arg realsense_enable)">
+    <xacro:sensor_d435 name="realsense_d435" topics_ns="realsense_d435" parent="base_link" publish_pointcloud="$(arg pointcloud_enable)" >
+      <origin xyz="0.077 0 0" rpy="0 0 0" />
+    </xacro:sensor_d435>
+  </xacro:if>
   <!-- BOARDS -->
-  <xacro:include filename="$(find jetbot_diff_drive)/urdf/includes/parts/boards.xacro" />
+  <xacro:pcb />
 </robot>

Commit message: added rplidar for rviz and gazebo

File: urdf/includes.xacro (robot description, xacro)
@@ -34,3 +34,6 @@
   <xacro:include filename="$(find jetbot_diff_drive)/urdf/includes/parts/sensors/realsense/_d435.urdf.xacro" />
   <!-- Intel Realsense Macro -->
+  <!-- RPLidar -->
+  <xacro:include filename="$(find jetbot_diff_drive)/urdf/includes/parts/sensors/laser/laser.urdf.xacro" />
+  <!-- RPLidar -->
 </robot>

File: urdf/includes/gazebo/jetbot.gazebo.xacro (robot description, xacro)
@@ -7,4 +7,33 @@
     </plugin>
   </gazebo>
+  <!-- Gazebo Plugin for IMU -->
+  <!--gazebo>
+    <plugin name="imu_plugin" filename="libgazebo_ros_imu.so">
+      <alwaysOn>true</alwaysOn>
+      <bodyName>imu_link</bodyName>
+      <frameName>imu_link</frameName>
+      <topicName>imu</topicName>
+      <serviceName>imu_service</serviceName>
+      <gaussianNoise>0.0</gaussianNoise>
+      <updateRate>200</updateRate>
+      <imu>
+        <noise>
+          <type>gaussian</type>
+          <rate>
+            <mean>0.0</mean>
+            <stddev>2e-4</stddev>
+            <bias_mean>0.0000075</bias_mean>
+            <bias_stddev>0.0000008</bias_stddev>
+          </rate>
+          <accel>
+            <mean>0.0</mean>
+            <stddev>1.7e-2</stddev>
+            <bias_mean>0.1</bias_mean>
+            <bias_stddev>0.001</bias_stddev>
+          </accel>
+        </noise>
+      </imu>
+    </plugin>
+  </gazebo-->
   <!--Gazebo Camera Plugin-->
   <gazebo reference="camera_lens">

File: urdf/includes/materials/materials.xacro (robot description, xacro)
@@ -22,3 +22,6 @@
     <color rgba="0.1 0.3 0.1 0.8"/>
   </material>
+  <material name="dark">
+    <color rgba="0.3 0.3 0.3 1.0"/>
+  </material>
 </robot>

File: urdf/includes/parts/chassis.xacro (robot description, xacro)
@@ -9,4 +9,5 @@
   <!-- CHASSIS (body) -->
   <xacro:macro name="chassis" >
+  <link name="odom" />
   <link name="base_link">
     <visual>
@@ -25,4 +26,10 @@
     <xacro:cuboid_inertia mass="0.6" x="${base_len}" y="${base_width}" z="${base_height}" />
   </link>
+  <!-- Joint to connect base_footprint with base_link -->
+  <joint name="odom_joint" type="fixed">
+    <origin xyz="0 0 0" rpy="0 0 0" />
+    <parent link="odom"/>
+    <child link="base_link" />
+  </joint>
   </xacro:macro>
   <!-- CHASSIS (body) -->

File: urdf/jetbot.xacro (robot description, xacro)
@@ -1,7 +1,10 @@
 <?xml version="1.0"?>
 <robot xmlns:xacro="http://www.ros.org/wiki/xacro" name="jetbot">
-  <!-- Xacro arguments for nominal use -->
+  <!-- Xacro arguments for depth camera use -->
   <xacro:arg name="realsense_enable" default="true" />
   <xacro:arg name="pointcloud_enable" default="true" />
+  <!-- Xacro arguments for depth lidar use -->
+  <xacro:arg name="lidar_enable" default="true" />
+  <xacro:arg name="visualize_laser" default="true" />
   <!-- All Neccesary Header Files, Macros and Constants -->
   <xacro:include filename="$(find jetbot_diff_drive)/urdf/includes.xacro" />
@@ -24,4 +27,6 @@
   <!-- MONOCULAR CAMERA -->
   <xacro:camera />
+  <!-- BOARDS -->
+  <xacro:pcb />
   <!-- REALSENSE CAMERA -->
   <xacro:if value="$(arg realsense_enable)">
@@ -30,5 +35,9 @@
     </xacro:sensor_d435>
   </xacro:if>
-  <!-- BOARDS -->
-  <xacro:pcb />
+  <!-- RPLIDAR LASER -->
+  <xacro:if value="$(arg lidar_enable)" >
+    <xacro:sensor_rplidar name="rplidar" topic_ns="rplidar" parent="pcb_boards" visualize_laser="$(arg visualize_laser)" >
+      <origin xyz="0 0 0.058" rpy="0 0 0" />
+    </xacro:sensor_rplidar >
+  </xacro:if>
 </robot>

Commit message: hector imu plugin with rviz and gazebo working

File: urdf/includes.xacro (robot description, xacro)
@@ -37,3 +37,12 @@
   <xacro:include filename="$(find jetbot_diff_drive)/urdf/includes/parts/sensors/laser/laser.urdf.xacro" />
   <!-- RPLidar -->
+  <!-- Sonar -->
+  <!--xacro:include filename="$(find jetbot_diff_drive)/urdf/includes/parts/sensors/sonar/hcsr04.urdf.xacro" /-->
+  <!-- Sonar -->
+  <!-- IMU -->
+  <xacro:include filename="$(find jetbot_diff_drive)/urdf/includes/parts/sensors/imu/bno055.urdf.xacro" />
+  <!-- IMU -->
+  <!-- GPS -->
+  <!--xacro:include filename="$(find jetbot_diff_drive)/urdf/includes/parts/sensors/gps/gps_mtk3339.urdf.xacro" /-->
+  <!-- GPS -->
 </robot>

File: urdf/includes/gazebo/jetbot.gazebo.xacro (robot description, xacro)
@@ -7,33 +7,4 @@
     </plugin>
   </gazebo>
-  <!-- Gazebo Plugin for IMU -->
-  <!--gazebo>
-    <plugin name="imu_plugin" filename="libgazebo_ros_imu.so">
-      <alwaysOn>true</alwaysOn>
-      <bodyName>imu_link</bodyName>
-      <frameName>imu_link</frameName>
-      <topicName>imu</topicName>
-      <serviceName>imu_service</serviceName>
-      <gaussianNoise>0.0</gaussianNoise>
-      <updateRate>200</updateRate>
-      <imu>
-        <noise>
-          <type>gaussian</type>
-          <rate>
-            <mean>0.0</mean>
-            <stddev>2e-4</stddev>
-            <bias_mean>0.0000075</bias_mean>
-            <bias_stddev>0.0000008</bias_stddev>
-          </rate>
-          <accel>
-            <mean>0.0</mean>
-            <stddev>1.7e-2</stddev>
-            <bias_mean>0.1</bias_mean>
-            <bias_stddev>0.001</bias_stddev>
-          </accel>
-        </noise>
-      </imu>
-    </plugin>
-  </gazebo-->
   <!--Gazebo Camera Plugin-->
   <gazebo reference="camera_lens">
@@ -77,4 +48,15 @@
   </gazebo>
   <!-- Hardcoding all the links here for colors -->
+  <gazebo reference="odom">
+    <mu1>0.2</mu1>
+    <mu2>0.2</mu2>
+    <material>Gazebo/White</material>
+  </gazebo>
+  <!-- Base Footprint Link -->
+  <gazebo reference="base_footprint">
+    <mu1>0.2</mu1>
+    <mu2>0.2</mu2>
+    <material>Gazebo/White</material>
+  </gazebo>
   <!-- Base Link -->
   <gazebo reference="base_link">
@@ -224,4 +206,9 @@
     <material>Gazebo/GreenTransparent</material>
   </gazebo>
+  <gazebo reference="bno055_base">
+    <mu1>0.2</mu1>
+    <mu2>0.2</mu2>
+    <material>Gazebo/Yellow</material>
+  </gazebo>
   <!-- Hardcoding all the links here for colors -->
 </robot>

File: urdf/includes/materials/materials.xacro (robot description, xacro)
@@ -1,4 +1,7 @@
 <?xml version="1.0"?>
 <robot>
+  <material name="yellow">
+    <color rgba="1 1 0 1"/>
+  </material>
   <material name="black">
     <color rgba="0 0 0 1"/>

File: urdf/includes/parts/chassis.xacro (robot description, xacro)
@@ -10,4 +10,5 @@
   <xacro:macro name="chassis" >
   <link name="odom" />
+  <link name="base_footprint" />
   <link name="base_link">
     <visual>
@@ -26,9 +27,13 @@
     <xacro:cuboid_inertia mass="0.6" x="${base_len}" y="${base_width}" z="${base_height}" />
   </link>
-  <!-- Joint to connect base_footprint with base_link -->
+  <!-- Joint to connect base_link with base_footprint -->
+  <joint name="base_footprint_joint" type="fixed">
+    <parent link="base_footprint"/>
+    <child link="base_link" />
+  </joint>
+  <!-- Joint to connect base_footprint with odom -->
   <joint name="odom_joint" type="fixed">
-    <origin xyz="0 0 0" rpy="0 0 0" />
     <parent link="odom"/>
-    <child link="base_link" />
+    <child link="base_footprint" />
   </joint>
   </xacro:macro>

File: urdf/jetbot.xacro (robot description, xacro)
@@ -41,3 +41,9 @@
     </xacro:sensor_rplidar >
   </xacro:if>
+  <!-- RPLIDAR LASER -->
+  <xacro:if value="$(arg imu_enable)" >
+    <xacro:sensor_imu name="bno055_imu" topic_ns="bno055_imu" parent="pcb_boards" >
+      <origin xyz="0 0 0.0275" rpy="0 0 0" />
+    </xacro:sensor_imu>
+  </xacro:if>
 </robot>
