Commit message: added more sensors to simulation sonar, odom, gps, imu

File: urdf/includes.xacro (robot description, xacro)
@@ -37,12 +37,12 @@
   <xacro:include filename="$(find jetbot_diff_drive)/urdf/includes/parts/sensors/laser/laser.urdf.xacro" />
   <!-- RPLidar -->
-  <!-- Sonar -->
-  <!--xacro:include filename="$(find jetbot_diff_drive)/urdf/includes/parts/sensors/sonar/hcsr04.urdf.xacro" /-->
-  <!-- Sonar -->
   <!-- IMU -->
   <xacro:include filename="$(find jetbot_diff_drive)/urdf/includes/parts/sensors/imu/bno055.urdf.xacro" />
   <!-- IMU -->
   <!-- GPS -->
-  <!--xacro:include filename="$(find jetbot_diff_drive)/urdf/includes/parts/sensors/gps/gps_mtk3339.urdf.xacro" /-->
+  <xacro:include filename="$(find jetbot_diff_drive)/urdf/includes/parts/sensors/gps/mtk3339.urdf.xacro" />
   <!-- GPS -->
+  <!-- Sonar -->
+  <xacro:include filename="$(find jetbot_diff_drive)/urdf/includes/parts/sensors/sonar/hcsr04.urdf.xacro" />
+  <!-- SOnar -->
 </robot>

File: urdf/includes/gazebo/inertias.xacro (robot description, xacro)
@@ -16,21 +16,30 @@
   <!-- cuboid inertia -->
   <xacro:macro name="cuboid_inertia" params="mass x y z">
+    <inertial>
+      <mass value="${mass}"/>
       <inertia  ixx="${mass*(y*y+z*z)/12}" ixy = "0" ixz = "0"
                 iyy="${mass*(x*x+z*z)/12}" iyz = "0"
-                izz="${mass*(x*x+z*z)/12}" />
+                izz="${mass*(x*x+y*y)/12}" />
+    </inertial>
   </xacro:macro>
   <!-- cuboid inertia -->
   <!-- sphere inertia -->
   <xacro:macro name="sphere_inertia" params="mass r">
-    <inertia  ixx="${2*mass*r*r/5}" ixy = "0" ixz = "0"
-              iyy="${2*mass*r*r/5}" iyz = "0"
-              izz="${2*mass*r*r/5}" />
+    <inertial>
+      <mass value="${mass}"/>
+      <inertia  ixx="${2*mass*r*r/5}" ixy = "0" ixz = "0"
+                iyy="${2*mass*r*r/5}" iyz = "0"
+                izz="${2*mass*r*r/5}" />
+    </inertial>
   </xacro:macro>
   <!-- sphere inertia -->
   <!-- cylinder inertia -->
   <xacro:macro name="cylinder_inertia" params="mass r h">
-    <inertia  ixx="${mass*(3*r*r+h*h)/12}" ixy = "0" ixz = "0"
-              iyy="${mass*(3*r*r+h*h)/12}" iyz = "0"
-              izz="${mass*r*r/2}" />
+    <inertial>
+      <mass value="${mass}"/>
+      <inertia  ixx="${mass*(3*r*r+h*h)/12}" ixy = "0" ixz = "0"
+                iyy="${mass*(3*r*r+h*h)/12}" iyz = "0"
+                izz="${mass*r*r/2}" />
+    </inertial>
   </xacro:macro>
   <!-- cylinder inertia -->

File: urdf/includes/gazebo/jetbot.gazebo.xacro (robot description, xacro)
@@ -47,167 +47,152 @@
     </sensor>
   </gazebo>
+   <gazebo>
+    <plugin name="p3d_base_controller" filename="libgazebo_ros_p3d.so">
+      <rpyOffsets>0 0 0</rpyOffsets>
+      <xyzOffsets>0 0 0</xyzOffsets>
+      <frameName>base_footprint</frameName>
+      <gaussianNoise>0.01</gaussianNoise>
+      <topicName>gazebo_robot_pose</topicName>
+      <bodyName>base_link</bodyName>
+      <updateRate>50.0</updateRate>
+      <alwaysOn>true</alwaysOn>
+    </plugin>
+  </gazebo>
   <!-- Hardcoding all the links here for colors -->
   <gazebo reference="odom">
-    <mu1>0.2</mu1>
-    <mu2>0.2</mu2>
     <material>Gazebo/White</material>
   </gazebo>
   <!-- Base Footprint Link -->
   <gazebo reference="base_footprint">
-    <mu1>0.2</mu1>
-    <mu2>0.2</mu2>
     <material>Gazebo/White</material>
   </gazebo>
   <!-- Base Link -->
   <gazebo reference="base_link">
-    <mu1>0.2</mu1>
-    <mu2>0.2</mu2>
     <material>Gazebo/BlueTransparent</material>
   </gazebo>
   <!-- Shaft Link -->
   <gazebo reference="lt_wheel_shaft">
-    <mu1>0.2</mu1>
-    <mu2>0.2</mu2>
     <material>Gazebo/White</material>
   </gazebo>
   <gazebo reference="rt_wheel_shaft">
-    <mu1>0.2</mu1>
-    <mu2>0.2</mu2>
     <material>Gazebo/White</material>
   </gazebo>
   <!-- Wheels Links -->
   <gazebo reference="lt_wheelc">
-    <mu1>0.2</mu1>
-    <mu2>0.2</mu2>
     <material>Gazebo/White</material>
   </gazebo>
   <gazebo reference="rt_wheelc">
-    <mu1>0.2</mu1>
-    <mu2>0.2</mu2>
     <material>Gazebo/White</material>
   </gazebo>
   <gazebo reference="lt_wheel">
-    <mu1>0.2</mu1>
-    <mu2>0.2</mu2>
+    <mu1>1.16</mu1>
+    <mu2>1.16</mu2>
     <material>Gazebo/Black</material>
   </gazebo>
   <gazebo reference="rt_wheel">
-    <mu1>0.2</mu1>
-    <mu2>0.2</mu2>
+    <mu1>1.16</mu1>
+    <mu2>1.16</mu2>
     <material>Gazebo/Black</material>
   </gazebo>
   <!-- Caster Links -->
   <gazebo reference="front_caster_lt_cyl">
-    <mu1>0.2</mu1>
-    <mu2>0.2</mu2>
     <material>Gazebo/White</material>
   </gazebo>
   <gazebo reference="front_caster_rt_cyl">
-    <mu1>0.2</mu1>
-    <mu2>0.2</mu2>
     <material>Gazebo/White</material>
   </gazebo>
   <gazebo reference="back_caster_lt_cyl">
-    <mu1>0.2</mu1>
-    <mu2>0.2</mu2>
     <material>Gazebo/White</material>
   </gazebo>
   <gazebo reference="back_caster_rt_cyl">
-    <mu1>0.2</mu1>
-    <mu2>0.2</mu2>
     <material>Gazebo/White</material>
   </gazebo>
   <gazebo reference="front_caster_base">
-    <mu1>0.2</mu1>
-    <mu2>0.2</mu2>
     <material>Gazebo/White</material>
   </gazebo>
   <gazebo reference="back_caster_base">
-    <mu1>0.2</mu1>
-    <mu2>0.2</mu2>
     <material>Gazebo/White</material>
   </gazebo>
   <gazebo reference="front_caster">
-    <mu1>0.2</mu1>
-    <mu2>0.2</mu2>
+    <mu1>0.01</mu1>
+    <mu2>0.01</mu2>
     <material>Gazebo/Grey</material>
   </gazebo>
   <gazebo reference="back_caster">
-    <mu1>0.2</mu1>
-    <mu2>0.2</mu2>
+    <mu1>0.01</mu1>
+    <mu2>0.01</mu2>
     <material>Gazebo/Grey</material>
   </gazebo>
   <!-- Antenna Links -->
   <gazebo reference="lt_antenna">
-    <mu1>0.2</mu1>
-    <mu2>0.2</mu2>
     <material>Gazebo/Black</material>
   </gazebo>
   <gazebo reference="rt_antenna">
-    <mu1>0.2</mu1>
-    <mu2>0.2</mu2>
     <material>Gazebo/Black</material>
   </gazebo>
   <gazebo reference="lt_antenna_top">
-    <mu1>0.2</mu1>
-    <mu2>0.2</mu2>
     <material>Gazebo/Black</material>
   </gazebo>
   <gazebo reference="rt_antenna_top">
-    <mu1>0.2</mu1>
-    <mu2>0.2</mu2>
     <material>Gazebo/Black</material>
   </gazebo>
   <!-- Camera Links -->
   <gazebo reference="camera_mount_base">
-    <mu1>0.2</mu1>
-    <mu2>0.2</mu2>
     <material>Gazebo/BlueTransparent</material>
   </gazebo>
   <gazebo reference="camera_mount_over">
-    <mu1>0.2</mu1>
-    <mu2>0.2</mu2>
     <material>Gazebo/BlueTransparent</material>
   </gazebo>
   <gazebo reference="camera_mount_angled">
-    <mu1>0.2</mu1>
-    <mu2>0.2</mu2>
     <material>Gazebo/BlueTransparent</material>
   </gazebo>
   <gazebo reference="camera_screen_base">
-    <mu1>0.2</mu1>
-    <mu2>0.2</mu2>
     <material>Gazebo/SkyBlue</material>
   </gazebo>
   <gazebo reference="camera_pcb_base">
-    <mu1>0.2</mu1>
-    <mu2>0.2</mu2>
     <material>Gazebo/Black</material>
   </gazebo>
   <gazebo reference="camera_lens_body">
-    <mu1>0.2</mu1>
-    <mu2>0.2</mu2>
     <material>Gazebo/Black</material>
   </gazebo>
   <gazebo reference="camera_lens_body_out">
-    <mu1>0.2</mu1>
-    <mu2>0.2</mu2>
     <material>Gazebo/Black</material>
   </gazebo>
   <gazebo reference="camera_lens">
-    <mu1>0.2</mu1>
-    <mu2>0.2</mu2>
     <material>Gazebo/GreyTransparent</material>
   </gazebo>
   <!-- Jetson Nano and Motor Driver Board -->
   <gazebo reference="pcb_boards">
-    <mu1>0.2</mu1>
-    <mu2>0.2</mu2>
     <material>Gazebo/GreenTransparent</material>
   </gazebo>
   <gazebo reference="bno055_base">
-    <mu1>0.2</mu1>
-    <mu2>0.2</mu2>
     <material>Gazebo/Yellow</material>
+  </gazebo>
+  <gazebo reference="mtk3339_link">
+    <material>Gazebo/Yellow</material>
+  </gazebo>
+  <gazebo reference="back_rt45_sonar_8_link">
+    <material>Gazebo/Purple</material>
+  </gazebo>
+  <gazebo reference="back_sonar_7_link">
+    <material>Gazebo/Purple</material>
+  </gazebo>
+  <gazebo reference="back_lt45_sonar_6_link">
+    <material>Gazebo/Purple</material>
+  </gazebo>
+    <gazebo reference="back_lt_sonar_5_link">
+    <material>Gazebo/Purple</material>
+  </gazebo>
+    <gazebo reference="front_lt45_sonar_4_link">
+    <material>Gazebo/Purple</material>
+  </gazebo>
+    <gazebo reference="front_sonar_3_link">
+    <material>Gazebo/Purple</material>
+  </gazebo>
+    <gazebo reference="front_rt45_sonar_2_link">
+    <material>Gazebo/Purple</material>
+  </gazebo>
+    <gazebo reference="back_rt_sonar_1_link">
+    <material>Gazebo/Purple</material>
   </gazebo>
   <!-- Hardcoding all the links here for colors -->

File: urdf/includes/gazebo/transmission.xacro (robot description, xacro)
@@ -6,4 +6,5 @@
       <type>transmission_interface/SimpleTransmission</type>
       <actuator name="${prefix}_${suffix}_motor">
+        <hardwareInterface>hardware_interface/VelocityJointInterface</hardwareInterface>
         <mechanicalReduction>1</mechanicalReduction>
       </actuator>

File: urdf/includes/materials/materials.xacro (robot description, xacro)
@@ -1,4 +1,7 @@
 <?xml version="1.0"?>
 <robot>
+  <material name="purple">
+    <color rgba="0.5 0 0.7 1"/>
+  </material>
   <material name="yellow">
     <color rgba="1 1 0 1"/>

File: urdf/includes/parts/antenna.xacro (robot description, xacro)
@@ -5,4 +5,8 @@
   <xacro:property name="antenna_r" value="0.005" />
   <xacro:property name="antenna_x" value="-0.645" />
+  <xacro:property name="antenna_body_mass" value="0.01" />
+  <xacro:property name="antenna_top_mass" value="0.000007" />
+  <!--xacro:property name="antenna_body_mass" value="0.6" />
+  <xacro:property name="antenna_top_mass" value="0.06" /-->
   <!-- Antenna constants -->
   <!-- Inertia Macros -->
@@ -25,5 +29,5 @@
       </geometry>
     </collision>
-    <xacro:cylinder_inertia mass="0.6" r="${antenna_r}" h="${antenna_len}" />
+    <xacro:cylinder_inertia mass="${antenna_body_mass}" r="${antenna_r}" h="${antenna_len}" />
   </link>
   <joint name="base_${prefix}_antenna_joint" type="fixed">
@@ -44,5 +48,5 @@
       </geometry>
     </collision>
-    <xacro:sphere_inertia mass="0.06" r="${antenna_r}" />
+    <xacro:sphere_inertia mass="${antenna_top_mass}" r="${antenna_r}" />
   </link>
   <joint name="${prefix}_antenna_top_joint" type="fixed">

File: urdf/includes/parts/boards.xacro (robot description, xacro)
@@ -5,4 +5,6 @@
   <xacro:property name="box_width" value="0.08" />
   <xacro:property name="box_height" value="0.055" />
+  <xacro:property name="box_mass" value="0.3645" />
+  <!--xacro:property name="box_mass" value="0.6" /-->
   <!-- Motor driver and PCB constants -->
   <!-- Inertias Macros -->
@@ -23,5 +25,5 @@
       </geometry>
     </collision>
-    <xacro:cuboid_inertia mass="0.6" x="${box_len}" y="${box_width}" z="${box_height}" />
+    <xacro:cuboid_inertia mass="${box_mass}" x="${box_len}" y="${box_width}" z="${box_height}" />
   </link>
   <joint name="base_nano_joint" type="fixed">

File: urdf/includes/parts/camera.xacro (robot description, xacro)
@@ -4,6 +4,17 @@
 <xacro:include filename="$(find jetbot_diff_drive)/urdf/includes/gazebo/inertias.xacro" />
 <!-- Inertias Macros -->
+<xacro:property name="camera_mount_base_mass" value="0.01" />
+<xacro:property name="camera_mount_over_mass" value="0.005" />
+<xacro:property name="camera_mount_angled_mass" value="0.0034" />
+<xacro:property name="camera_screen_base_mass" value="0.0017" />
+<xacro:property name="camera_pcb_base" value="0.00376" />
+<xacro:property name="camera_lens_body" value="0.000089" />
+<xacro:property name="camera_lens_body_out" value="0.0049" />
+<xacro:property name="camera_lens" value="0.000009" />
+<!--xacro:property name="camera_pcb_base" value="0.6" />
+<xacro:property name="camera_lens_body" value="0.6" />
+<xacro:property name="camera_lens_body_out" value="0.6" />
+<xacro:property name="camera_lens" value="0.6" /-->
 <!-- CAMERA -->
- <xacro:macro name="camera" >
   <link name="camera_mount_base">
     <visual>
@@ -18,5 +29,5 @@
       </geometry>
     </collision>
-    <xacro:cuboid_inertia mass="0.009" x="0.01" y="0.04" z="0.002" />
+    <xacro:cuboid_inertia mass="${camera_mount_base_mass}" x="0.01" y="0.04" z="0.002" />
   </link>
   <joint name="camera_mount_base_joint" type="fixed">
@@ -39,5 +50,5 @@
       </geometry>
     </collision>
-    <xacro:cuboid_inertia mass="0.009" x="0.03" y="0.04" z="0.002"/>
+    <xacro:cuboid_inertia mass="${camera_mount_over_mass}" x="0.03" y="0.04" z="0.002"/>
   </link>
   <joint name="camera_mount_over_joint" type="fixed">
@@ -60,10 +71,10 @@
       </geometry>
     </collision>
-    <xacro:cuboid_inertia mass="0.009" x="0.025" y="0.025" z="0.002" />
+    <xacro:cuboid_inertia mass="${camera_mount_angled_mass}" x="0.025" y="0.025" z="0.002" />
   </link>
   <joint name="camera_mount_angled_joint" type="fixed">
     <parent link="camera_mount_over"/>
     <child link="camera_mount_angled"/>
-    <origin rpy="0 0.24 0" xyz="0.003 0 0.027"/>
+    <origin rpy="0 0.463647609 0" xyz="0.0055 0 0.025"/>
   </joint>
   <link name="camera_screen_base">
@@ -81,5 +92,5 @@
       </geometry>
     </collision>
-    <xacro:cuboid_inertia mass="0.009" x="0.025" y="0.025" z="0.004" />
+    <xacro:cuboid_inertia mass="${camera_screen_base_mass}" x="0.025" y="0.025" z="0.004" />
   </link>
   <joint name="camera_mount_screen_joint" type="fixed">
@@ -102,5 +113,5 @@
       </geometry>
     </collision>
-    <xacro:cuboid_inertia mass="0.009" x="0.013" y="0.013" z="0.004" />
+    <xacro:cuboid_inertia mass="${camera_pcb_base_mass}" x="0.013" y="0.013" z="0.004" />
   </link>
   <joint name="camera_pcb_base_joint" type="fixed">
@@ -123,5 +134,5 @@
       </geometry>
     </collision>
-    <xacro:cylinder_inertia mass="0.022" r="0.006" h="0.01" />
+    <xacro:cylinder_inertia mass="${camera_lens_body_mass}" r="0.006" h="0.01" />
   </link>
   <joint name="camera_lens_body_joint" type="fixed">
@@ -144,5 +155,5 @@
       </geometry>
     </collision>
-    <xacro:cylinder_inertia mass="0.009" r="0.0075" h="0.003"/>
+    <xacro:cylinder_inertia mass="${camera_lens_body_out_mass}" r="0.0075" h="0.003"/>
   </link>
  <joint name="camera_lens_body_out_joint" type="fixed">
@@ -165,5 +176,5 @@
       </geometry>
     </collision>
-    <xacro:sphere_inertia mass="0.006" r="0.005" />
+    <xacro:sphere_inertia mass="${camera_lens_mass}" r="0.005" />
   </link>
  <joint name="camera_lens_joint" type="fixed">
@@ -172,4 +183,3 @@
     <origin xyz="-0.001 0 0"/>
   </joint>
-  </xacro:macro>
 </robot>

File: urdf/includes/parts/chassis.xacro (robot description, xacro)
@@ -6,4 +6,6 @@
   <xacro:property name="base_height" value="0.035"/>
   <xacro:property name="base_z_offset" value="0.013"/>
+  <xacro:property name="base_mass" value="0.045" />
+  <!--xacro:property name="base_mass" value="0.6" /-->
   <!-- Chassis constants -->
   <!-- CHASSIS (body) -->
@@ -25,5 +27,5 @@
       </geometry>
     </collision>
-    <xacro:cuboid_inertia mass="0.6" x="${base_len}" y="${base_width}" z="${base_height}" />
+    <xacro:cuboid_inertia mass="${base_mass}" x="${base_len}" y="${base_width}" z="${base_height}" />
   </link>
   <!-- Joint to connect base_link with base_footprint -->

File: urdf/includes/parts/sensors/imu/bno055.urdf.xacro (robot description, xacro)
@@ -13,5 +13,5 @@
   <!-- IMU BNO055 -->
   <xacro:macro name="sensor_imu" params="name topic_ns:=bno055 parent *origin">
-    <joint name="imu_joint" type="fixed">
+    <joint name="{name}_joint" type="fixed">
       <parent link="${parent}"/>
       <child link="${name}_base"/>
@@ -20,5 +20,5 @@
     <link name="${name}_base">
       <visual>
-        <origin xyz="-${bno_width/2} ${bno_height/2} -${bno_depth/2}" rpy="${pi/2} 0 0"/>
+        <origin xyz="-${bno_width/2} ${bno_height/2} 0" rpy="${pi/2} 0 0"/>
         <geometry>
           <mesh filename="package://jetbot_diff_drive/meshes/imu/bno055.stl" scale="0.001 0.001 0.001"/>
@@ -27,5 +27,5 @@
       </visual>
       <collision>
-        <origin xyz="0 0 0" rpy="0 0 0"/>
+        <origin xyz="0 0 ${bno_depth/2}" rpy="0 0 0"/>
         <geometry>
           <box size="${bno_width} ${bno_height} ${bno_depth}"/>

File: urdf/includes/parts/wheels/caster.xacro (robot description, xacro)
@@ -8,4 +8,7 @@
   <xacro:property name="caster_zoffset" value="-0.0097" />
   <xacro:property name="caster_ball" value="0.005" />
+  <xacro:property name="caster_minicyl_mass" value="0.0001" />
+  <xacro:property name="caster_cyl_mass" value="0.001" />
+  <xacro:property name="caster_ball_mass" value="0.02" />
   <!-- Caster Ball constants -->
   <!-- Inertia Macro -->
@@ -26,5 +29,5 @@
       </geometry>
     </collision>
-    <xacro:cylinder_inertia mass="0.6" r="${caster_cyl_r/3.75}" h="${caster_cyl_len}" />
+    <xacro:cylinder_inertia mass="${caster_minicyl_mass}" r="${caster_cyl_r/3.75}" h="${caster_cyl_len}" />
   </link>
   <joint name="${prefix}_caster_${suffix}_cyl_joint" type="fixed">
@@ -49,5 +52,5 @@
       </geometry>
     </collision>
-    <xacro:cylinder_inertia mass="0.6" r="${caster_cyl_r}" h="${caster_cyl_len}" />
+    <xacro:cylinder_inertia mass="${caster_cyl_mass}" r="${caster_cyl_r}" h="${caster_cyl_len}" />
   </link>
   <joint name="base_${prefix}_caster_joint" type="fixed">
@@ -70,5 +73,5 @@
       </geometry>
     </collision>
-    <xacro:sphere_inertia mass="0.6" r="${caster_ball}" />
+    <xacro:sphere_inertia mass="${caster_ball_mass}" r="${caster_ball}" />
   </link>
   <joint name="${prefix}_caster_joint" type="fixed">

File: urdf/includes/parts/wheels/wheel.xacro (robot description, xacro)
@@ -8,4 +8,10 @@
   <xacro:property name="wheelc_len" value="0.015" />
   <xacro:property name="wheelc_r" value = "0.026" />
+  <xacro:property name="wheel_shaft_mass" value = "0.0028" />
+  <xacro:property name="wheelc_mass" value = "0.0272" />
+  <xacro:property name="wheel_mass" value = "0.0181" />
+  <!--xacro:property name="wheel_shaft_mass" value="0.6" />
+  <xacro:property name="wheelc_mass" value="0.6" />
+  <xacro:property name="wheel_mass" value="0.6" /-->
   <!-- Wheel constants -->
   <!-- Inertia Macro -->
@@ -28,5 +34,5 @@
       </geometry>
     </collision>
-    <xacro:inertia mass="0.6" />
+    <xacro:cylinder_inertia mass="${wheel_shaft_mass}" r="${shaft_r}" h="${shaft_len}"/>
   </link>
   <joint name="base_${prefix}_wheel_shaft_joint" type="fixed">
@@ -51,4 +57,5 @@
     </collision>
     <xacro:inertia mass="0.6" />
+    <!--xacro:cylinder_inertia mass="${wheelc_mass}" r="${wheelc_r}" h="${wheelc_len}" /-->
   </link>
   <joint name="${prefix}_shaft_wheelc_joint" type="fixed">
@@ -72,4 +79,5 @@
     </collision>
     <xacro:inertia mass="0.6"/>
+    <!--xacro:cylinder_inertia mass="${wheel_mass}" r="${wheelc_r + 0.0065}" h="${wheelc_len}" /-->
   </link>
   <joint name="${prefix}_wheel_joint" type="continuous">

File: urdf/jetbot.xacro (robot description, xacro)
@@ -7,4 +7,10 @@
   <xacro:arg name="lidar_enable" default="true" />
   <xacro:arg name="visualize_laser" default="true" />
+  <!-- Xacro arguments for imu -->
+  <xacro:arg name="imu_enable" default="true" />
+  <!-- Xacro arguments for gps -->
+  <xacro:arg name="gps_enable" default="true" />
+  <!-- Xacro arguments for ultrasonic -->
+  <xacro:arg name="ultrasonic_enable" default="true" />
   <!-- All Neccesary Header Files, Macros and Constants -->
   <xacro:include filename="$(find jetbot_diff_drive)/urdf/includes.xacro" />
@@ -41,9 +47,42 @@
     </xacro:sensor_rplidar >
   </xacro:if>
-  <!-- RPLIDAR LASER -->
+  <!-- IMU -->
   <xacro:if value="$(arg imu_enable)" >
-    <xacro:sensor_imu name="bno055_imu" topic_ns="bno055_imu" parent="pcb_boards" >
+    <xacro:sensor_imu name="bno055" topic_ns="bno_imu" parent="pcb_boards" >
       <origin xyz="0 0 0.0275" rpy="0 0 0" />
     </xacro:sensor_imu>
   </xacro:if>
+  <!-- GPS -->
+  <xacro:if value="$(arg gps_enable)" >
+    <xacro:sensor_gps name="mtk3339" topic_ns="mtk_gps" parent="bno055_base" >
+      <origin xyz="-0.044 0 0" rpy="0 0 0" />
+    </xacro:sensor_gps>
+  </xacro:if>
+  <!-- Ultrasonic Sensors -->
+  <xacro:if value="$(arg ultrasonic_enable)" >
+    <xacro:sensor_sonar name="sonar_1" topic_ns="sonar_back_rt" prefix="back_rt" parent="base_link" >
+      <origin xyz="-${base_len/3.5} -${base_width/2} ${base_height/2}" rpy="0 0 -${pi/2}" />
+    </xacro:sensor_sonar>
+    <xacro:sensor_sonar name="sonar_2" topic_ns="sonar_front_rt45" prefix="front_rt45" parent="base_link" >
+      <origin xyz="${base_len/2} -${base_width/2} ${base_height+(base_z_offset)/2}" rpy="0 0 -${pi/4}" />
+    </xacro:sensor_sonar>
+    <xacro:sensor_sonar name="sonar_3" topic_ns="sonar_front" prefix="front" parent="camera_mount_over" >
+      <origin xyz="0 0 0" rpy="0 0 0" />
+    </xacro:sensor_sonar>
+    <xacro:sensor_sonar name="sonar_4" topic_ns="sonar_front_lt45" prefix="front_lt45" parent="base_link" >
+      <origin xyz="${base_len/2} ${base_width/2} ${base_height+(base_z_offset)/2}" rpy="0 0 ${pi/4}" />
+    </xacro:sensor_sonar>
+    <xacro:sensor_sonar name="sonar_5" topic_ns="sonar_back_lt" prefix="back_lt" parent="base_link" >
+      <origin xyz="-${base_len/3.5} ${base_width/2} ${base_height/2}" rpy="0 0 ${pi/2}" />
+    </xacro:sensor_sonar>
+    <xacro:sensor_sonar name="sonar_6" topic_ns="sonar_back_lt45" prefix="back_lt45" parent="base_link" >
+      <origin xyz="-${base_len/2} ${base_width/2} ${base_height+(base_z_offset)/2}" rpy="0 0 ${pi/2 + pi/4}" />
+    </xacro:sensor_sonar>
+    <xacro:sensor_sonar name="sonar_7" topic_ns="sonar_back" prefix="back" parent="base_link" >
+      <origin xyz="-${base_len/2} 0 ${base_height/2}" rpy="0 0 ${pi}" />
+    </xacro:sensor_sonar>
+    <xacro:sensor_sonar name="sonar_8" topic_ns="sonar_back_rt45" prefix="back_rt45" parent="base_link" >
+      <origin xyz="-${base_len/2} -${base_width/2} ${base_height+(base_z_offset)/2}" rpy="0 0 -${pi/2 + pi/4}" />
+    </xacro:sensor_sonar>
+  </xacro:if>
 </robot>
