Commit message: added a soccer ball to the world and improved camera angle

File: urdf/includes/parts/camera.xacro (robot description, xacro)
@@ -64,5 +64,5 @@
     <parent link="camera_mount_over"/>
     <child link="camera_mount_angled"/>
-    <origin rpy="0 0.463647609 0" xyz="0.0055 0 0.025"/>
+    <origin rpy="0 0.24 0" xyz="0.003 0 0.027"/>
   </joint>
   <link name="camera_screen_base">
